File: precise_ammeter/power_USB.kicad_sch (KiCad schematic)
At the start: 21 parts, among them J3 USB4110GFA, J5 XT30_Male, U10 TPS7A2450DBVR, U7 TPS7A2433DBVR, U8 TPS7A2450DBVR, U9 LMC7660

Commit message: dodano layout
Parts:
- removed C23: 2u2, Capacitor_SMD:C_0805_2012Metric_Pad1.18x1.45mm_HandSolder, symbol Device:C
- removed D1, D2: Green, LED_SMD:LED_0805_2012Metric_Pad1.15x1.40mm_HandSolder, symbol Device:LED
- removed J5: XT30_Male, Connector_AMASS:AMASS_XT30UPB-M_1x02_P5.0mm_Vertical, symbol Connector:Conn_01x02_Pin
- removed R26, R27: 1k, Resistor_SMD:R_0805_2012Metric_Pad1.20x1.40mm_HandSolder, symbol Device:R
- removed U10, U8: TPS7A2450DBVR, TPS7A2450DBVR:SOT_50DBVR, symbol TPS7A2450DBVR:TPS7A2450DBVR
- added C40, C41, C42, C43, C44, C45, C46: 2u2, Capacitor_SMD:C_0805_2012Metric_Pad1.18x1.45mm_HandSolder, symbol Device:C
- added C47: 10u, Capacitor_SMD:CP_Elec_4x5.4, symbol Device:C_Polarized
- added D10, D8, D9: Green, LED_SMD:LED_0805_2012Metric_Pad1.15x1.40mm_HandSolder, symbol Device:LED
- added R30, R31, R32: 1k, Resistor_SMD:R_0805_2012Metric_Pad1.20x1.40mm_HandSolder, symbol Device:R
- J3: footprint USB4100GFA:GCT_USB4110GFA -> USB4110GFA:GCT_USB4110GFA
- U7: footprint SOT23_DBV_TEX -> Package_TO_SOT_SMD:SOT-23-5_HandSoldering
Connections:
- net +3V3: now also R31.1
- net +5VA: now also C1.1, C22.1, C28.1, J3.A4/B9 (VBUS), J3.B4/A9 (VBUS), U7.1 (Vin), U7.3 (EN), U9.8 (V+), C40.1, C41.1, C42.1, C43.1, C44.1, C45.1, R30.1
- net -5VA: now also C25.1, C26.1, C46.1, R32.1
- net GND: now also C40.2, C41.2, C42.2, C43.2, C44.2, C45.2, C46.2, D10.2 (A), D8.1 (K), D9.1 (K)
- net at C24.1, U9.2 (CAP+): now also C47.1
- net at C24.2, U9.4 (CAP-): now also C47.2
- removed net +5V_U9: C26.1, C28.1, U9.8 (V+)
- removed net VBUS: C1.1, C22.1, C25.1, U7.1 (Vin), U7.3 (EN)
- new net: D10.1 (K), R32.2
- new net: D8.2 (A), R30.2
- new net: D9.2 (A), R31.2
- no-connect marks 8 -> 4
Other:
- note added: "USB 2.0 Type C"
- note removed: "USB 2.0 Type C for data transfer only"
- moved on the sheet: C1, C22, C24, C27, C28, C5, J3, R28, R29, U7, U9
