File: precise_ammeter/power_USB.kicad_sch (KiCad schematic)
At the start: 22 parts, among them J3 USB4110GFA, J5 XT30_Male, U10 TPS7A2450DBVR, U7 TPS7A2433DBVR, U8 TPS7A2450DBVR, U9 LMC7660

Commit message: jebane gowno
Parts:
- removed C39: 10u, Capacitor_SMD:CP_Elec_4x5.4, symbol Device:C_Polarized
Changed lines of the file:
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@@
 	)
 	(junction
-		(at 257.81 115.57)
-		(diameter 0)
-		(color 0 0 0 0)
-	)
-	(junction
 		(at 81.28 127)
 		(diameter 0)
@@
 	)
 	(junction
-		(at 257.81 125.73)
-		(diameter 0)
-		(color 0 0 0 0)
-	)
-	(junction
 		(at 100.33 181.61)
 		(diameter 0)
@@
 	(wire
 		(pts
-			(xy 270.51 115.57) (xy 257.81 115.57)
-		)
-		(stroke
-			(width 0)
-			(type default)
-		)
-	)
-	(wire
-		(pts
 			(xy 85.09 114.3) (xy 81.28 114.3)
 		)
@@
 	(wire
 		(pts
-			(xy 270.51 116.84) (xy 270.51 115.57)
-		)
-		(stroke
-			(width 0)
-			(type default)
-		)
-	)
-	(wire
-		(pts
 			(xy 210.82 46.99) (xy 207.01 46.99)
 		)
@@
 	(wire
 		(pts
-			(xy 270.51 124.46) (xy 270.51 125.73)
-		)
-		(stroke
-			(width 0)
-			(type default)
-		)
-	)
-	(wire
-		(pts
 			(xy 81.28 116.84) (xy 81.28 121.92)
 		)
@@
 	(wire
 		(pts
-			(xy 257.81 125.73) (xy 270.51 125.73)
-		)
-		(stroke
-			(width 0)
-			(type default)
-		)
-	)
-	(wire
-		(pts
 			(xy 60.96 181.61) (xy 60.96 176.53)
 		)
@@
 					(unit 1)
 				)
-			)
-		)
-	)
-	(symbol
-		(lib_id "Device:C_Polarized")
-		(at 270.51 120.65 0)
-		(unit 1)
-		(exclude_from_sim no)
-		(in_bom yes)
-		(on_board yes)
-		(dnp no)
-		(fields_autoplaced yes)
-		(property "Reference" "C39"
-			(at 274.32 118.4909 0)
-			(effects
-				(font
-					(size 1.27 1.27)
-				)
-				(justify left)
-			)
-		)
-		(property "Value" "10u"
-			(at 274.32 121.0309 0)
-			(effects
-				(font
-					(size 1.27 1.27)
-				)
-				(justify left)
-			)
-		)
-		(property "Footprint" "Capacitor_SMD:CP_Elec_4x5.4"
-			(at 271.4752 124.46 0)
-			(effects
-				(font
-					(size 1.27 1.27)
-				)
-				(hide yes)
-			)
-		)
-		(property "Datasheet" "~"
-			(at 270.51 120.65 0)
-			(effects
-				(font
-					(size 1.27 1.27)
-				)
-				(hide yes)
-			)
-		)
-		(property "Description" "Polarized capacitor"
-			(at 270.51 120.65 0)
-			(effects
-				(font
-					(size 1.27 1.27)
-				)
-				(hide yes)
-			)
-		)
-		(property "Product link" "EDH106M025S9BAA"
-			(at 270.51 120.65 0)
-			(effects
-				(font
-					(size 1.27 1.27)
-				)
-				(hide yes)
-			)
-		)
-		(pin "2"
-		)
-		(pin "1"
-		)
-		(instances
-			(project "precise_ammeter"
-				(path "/7da3b652-85ac-4caa-8d8d-9cad461e9c85/9e6d6147-95e6-4ef0-a238-5628802dd2a2"
-					(reference "C39")
-					(unit 1)
-				)

Commit message: Layout Done, DRC done
Parts:
- U7: footprint SOT23_DBV_TEX -> TPS7A2433DBVR:SOT23_DBV_TEX
Changed lines of the file:
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@@
 			)
 		)
-		(property "Footprint" "SOT23_DBV_TEX"
+		(property "Footprint" "TPS7A2433DBVR:SOT23_DBV_TEX"
 			(at 74.93 45.72 0)
 			(effects
