File: precise_ammeter/precise_ammeter.kicad_sch (KiCad schematic)
At the start: 2 parts, among them J1 Conn_01x01_Socket, J2 Conn_01x01_Socket

Commit message: dodano layout
Changed lines of the file:
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@@
 		)
 	)
-	(text_box "Subsheet provides:\n- USB lines for MCU (no +5V USB lines connected, only D+/-)\n- +3V3, +5VA and -5VA for MCU and analog section\n- Status LEDs"
+	(text_box "Subsheet provides:\n- USB lines for MCU\n- +3V3, +5VA and -5VA for MCU and analog section\n- Status LEDs"
 		(exclude_from_sim no)
 		(at 158.115 44.45 0)
